Commit message: fix_gcode_translation_bug

File: moveo_urdf/urdf/moveo_urdf1.urdf (robot description, URDF)
Before this commit: robot moveo_urdf, 8 links, 7 joints
Joints:
- joint moveo_joint4: limit lower=-1.3745 upper=4.5161 effort=10 velocity=100 -> lower=-0.08726 upper=0.08726 effort=10 velocity=100

File: moveo_urdf/urdf/moveo_urdf2.urdf (robot description, URDF)
Before this commit: robot moveo_urdf, 8 links, 7 joints
Joints:
- joint moveo_joint4: limit lower=-1.3745 upper=4.5161 effort=10 velocity=100 -> lower=3.05433 upper=3.22886 effort=10 velocity=100
