Commit message: change urdf and moveo_moveit_config

File: moveo_urdf/urdf/moveo_urdf.urdf (robot description, URDF)
Before this commit: robot moveo_urdf, 13 links, 12 joints
Links:
- removed link moveo_gripper_link1
- removed link moveo_gripper_link2
- removed link moveo_gripper_link3
- removed link moveo_gripper_link4
- removed link moveo_gripper_link5
- removed link moveo_gripper_link6
- added link end_effector_link, mass 0.0102853681251992; collision mesh filename=package://moveo_urdf/meshes/end_effector_link.STL; visual mesh filename=package://moveo_urdf/meshes/end_effector_link.STL
- link moveo_link1: mass 4.14596598503804 -> 4.14595797854913
- link moveo_link2: mass 1.90833274539581 -> 1.90837643765425
- link moveo_link3: mass 0.65464588761888 -> 0.654645252090226
- link moveo_link4: mass 0.612035593213448 -> 0.620570358159444
- link moveo_link5: mass 0.189731615639297 -> 0.21298004137125
Joints:
- removed joint moveo_gripper_joint1
- removed joint moveo_gripper_joint2
- removed joint moveo_gripper_joint3
- removed joint moveo_gripper_joint4
- removed joint moveo_gripper_joint5
- removed joint moveo_gripper_joint6
- added joint end_effector_joint: type fixed, parent moveo_link5, child end_effector_link, origin xyz=-0.040668 -0.001931 0.12926 rpy=0 0 0, axis 0 0 0
- joint moveo_joint1: axis 0 1 0 -> 0 0 1; limit lower=-1.5707 upper=1.5707 effort=5 velocity=1 -> lower=-1.7543 upper=1.7543 effort=10 velocity=100; origin xyz=0 0 0.066 rpy=-1.5708 0 -3.1139 -> xyz=0 0 0.0665 rpy=0 0 0
- joint moveo_joint2: axis 0 1 0 -> -0.99939 -0.035015 0; limit lower=-1.5707 upper=1.5707 effort=5 velocity=3 -> lower=-1.7543 upper=1.7543 effort=10 velocity=100; origin xyz=0 -0.1655 0 rpy=0 0.82923 1.5708 -> xyz=0 0 0.165 rpy=0 0 0
- joint moveo_joint3: axis 0.99962 0.0277 0 -> -0.99939 -0.035015 0; limit lower=-1.5707 upper=1.5707 effort=5 velocity=3 -> lower=-1.7543 upper=1.7543 effort=10 velocity=100; origin xyz=-4.4369E-05 0 -0.22112 rpy=-2.4002 -0.018711 1.5912 -> xyz=0.00099794 7.6228E-05 0.22112 rpy=0 0 0
- joint moveo_joint4: axis 0.025906 -0.9349 -0.35396 -> 0.00023378 -0.0066725 0.99998; limit lower=-3.1416 upper=3.1416 effort=5 velocity=3 -> lower=-1.7543 upper=1.7543 effort=10 velocity=100; origin xyz=-0.0022967 0.11898 0.045038 rpy=0 0 0 -> xyz=2.9924E-05 -0.00085408 0.128 rpy=0 0 0
- joint moveo_joint5: axis 0.00069194 1 0.00091055 -> -0.99935 -0.035919 0; limit lower=-1.5707 upper=1.5707 effort=5 velocity=3 -> lower=-1.7543 upper=1.7543 effort=10 velocity=100; origin xyz=-0.0024817 0.089559 0.033866 rpy=0.24894 -1.0009 1.4384 -> xyz=2.2209E-05 -0.00063389 0.094998 rpy=0 0 0

Commit message: change urdf and moveit_config

File: moveo_urdf/urdf/moveo_urdf.urdf (robot description, URDF)
Before this commit: robot moveo_urdf, 8 links, 7 joints
Links:
- removed link end_effector_link
- link moveo_link1: mass 4.14595797854913 -> 4.17940224565423
- link moveo_link2: mass 1.90837643765425 -> 1.91858407284866
- link moveo_link3: mass 0.654645252090226 -> 0.654645252090227
- link moveo_link4: mass 0.620570358159444 -> 0.623350768745705
- link moveo_link5: mass 0.21298004137125 -> 0.718210813715952
Joints:
- removed joint end_effector_joint
- joint moveo_joint1: limit lower=-1.7543 upper=1.7543 effort=10 velocity=100 -> lower=-1.745 upper=1.745 effort=10 velocity=100
- joint moveo_joint2: limit lower=-1.7543 upper=1.7543 effort=10 velocity=100 -> lower=-1.745 upper=1.745 effort=10 velocity=100
- joint moveo_joint3: limit lower=-1.7543 upper=1.7543 effort=10 velocity=100 -> lower=-1.745 upper=1.745 effort=10 velocity=100
- joint moveo_joint4: limit lower=-1.7543 upper=1.7543 effort=10 velocity=100 -> lower=-1.745 upper=1.745 effort=10 velocity=100
- joint moveo_joint5: limit lower=-1.7543 upper=1.7543 effort=10 velocity=100 -> lower=-1.745 upper=1.745 effort=10 velocity=100

Commit message: add nozzle to urdf and chage moveit_config

File: moveo_urdf/urdf/moveo_urdf.urdf (robot description, URDF)
Before this commit: robot moveo_urdf, 7 links, 6 joints
Joints:
- joint moveo_joint4: limit lower=-1.745 upper=1.745 effort=10 velocity=100 -> lower=-3.1416 upper=3.1416 effort=10 velocity=100

Commit message: fix bug can't draw trajectoryLine on rviz

File: moveo_urdf/urdf/moveo_urdf.urdf (robot description, URDF)
Before this commit: robot moveo_urdf, 7 links, 6 joints
Links:
- added link moveo_nozzle_link, mass 0.56075; collision mesh filename=package://moveo_urdf/meshes/moveo_nozzle_link.STL; visual mesh filename=package://moveo_urdf/meshes/moveo_nozzle_link.STL
- link moveo_link1: mass 4.17940224565423 -> 4.146
- link moveo_link2: mass 1.91858407284866 -> 1.9084
- link moveo_link3: mass 0.654645252090227 -> 0.65465
- link moveo_link4: mass 0.623350768745705 -> 0.61776
- link moveo_link5: mass 0.718210813715952 -> 0.15771
Joints:
- added joint moveo_nozzle_joint: type fixed, parent moveo_link5, child moveo_nozzle_link, origin xyz=0 4.6534E-05 0.041 rpy=1.5708 -0.0011359 -1.5349, axis 0 0 0
- joint moveo_joint4: limit lower=-3.1416 upper=3.1416 effort=10 velocity=100 -> lower=-3.1415926 upper=3.1415926 effort=10 velocity=100

Commit message: change target frame to nozzle

File: moveo_urdf/urdf/moveo_urdf.urdf (robot description, URDF)
Before this commit: robot moveo_urdf, 8 links, 7 joints
Links:
- link moveo_link1: mass 4.146 -> 4.20302329882691
- link moveo_link2: mass 1.9084 -> 1.91858407295863
- link moveo_link3: mass 0.65465 -> 0.654645252090227
- link moveo_link4: mass 0.61776 -> 0.623350768745701
- link moveo_link5: mass 0.15771 -> 0.157708113613127
- link moveo_nozzle_link: mass 0.56075 -> 0.562206501752102
Joints:
- joint moveo_joint1: limit lower=-1.745 upper=1.745 effort=10 velocity=100 -> lower=-1.746 upper=1.746 effort=10 velocity=100
- joint moveo_joint2: limit lower=-1.745 upper=1.745 effort=10 velocity=100 -> lower=-1.746 upper=1.746 effort=10 velocity=100
- joint moveo_joint3: limit lower=-1.745 upper=1.745 effort=10 velocity=100 -> lower=-1.746 upper=1.746 effort=10 velocity=100
- joint moveo_joint4: limit lower=-3.1415926 upper=3.1415926 effort=10 velocity=100 -> lower=-3.1416 upper=3.1416 effort=10 velocity=100
- joint moveo_joint5: limit lower=-1.745 upper=1.745 effort=10 velocity=100 -> lower=-1.746 upper=1.746 effort=10 velocity=100
- joint moveo_nozzle_joint: origin xyz=0 4.6534E-05 0.041 rpy=1.5708 -0.0011359 -1.5349 -> xyz=-0.012488 0.043982 0.10635 rpy=1.5697 0 0.035926

Commit message: update nozzle in urdf

File: moveo_urdf/urdf/moveo_urdf.urdf (robot description, URDF)
Before this commit: robot moveo_urdf, 8 links, 7 joints
Links:
- link moveo_link2: mass 1.91858407295863 -> 1.91858407296435
- link moveo_link4: mass 0.623350768745701 -> 0.623350768745695
- link moveo_link5: mass 0.157708113613127 -> 0.157708115385714
- link moveo_nozzle_link: mass 0.562206501752102 -> 0.560923295529705
Joints:
- joint moveo_nozzle_joint: origin xyz=-0.012488 0.043982 0.10635 rpy=1.5697 0 0.035926 -> xyz=-0.013528 0.072912 0.10432 rpy=1.5418 0 0.035926

Commit message: chang ompl planner to LazyPRM

File: moveo_urdf/urdf/moveo_urdf.urdf (robot description, URDF)
Before this commit: robot moveo_urdf, 8 links, 7 joints
Joints:
- joint moveo_joint1: limit lower=-1.746 upper=1.746 effort=10 velocity=100 -> lower=-2.150 upper=2.150 effort=10 velocity=100
- joint moveo_joint2: limit lower=-1.746 upper=1.746 effort=10 velocity=100 -> lower=-2.150 upper=2.150 effort=10 velocity=100
- joint moveo_joint3: limit lower=-1.746 upper=1.746 effort=10 velocity=100 -> lower=-2.150 upper=2.150 effort=10 velocity=100
- joint moveo_joint5: limit lower=-1.746 upper=1.746 effort=10 velocity=100 -> lower=-2.150 upper=2.150 effort=10 velocity=100

Commit message: gcode_translation_add_collision

File: moveo_urdf/urdf/moveo_urdf.urdf (robot description, URDF)
Before this commit: robot moveo_urdf, 8 links, 7 joints
Links:
- link base_link: mass 0.637576232475362 -> 0.637576232475361
- link moveo_link2: mass 1.91858407296435 -> 1.91858407297439
- link moveo_link3: mass 0.654645252090227 -> 0.648943927759347
- link moveo_nozzle_link: mass 0.560923295529705 -> 0.560923247976437
Joints:
- joint moveo_joint1: limit lower=-2.150 upper=2.150 effort=10 velocity=100 -> lower=-2.15 upper=2.15 effort=10 velocity=100
- joint moveo_joint2: axis -0.99939 -0.035015 0 -> -0.999386785928715 -0.0350150269323535 0; limit lower=-2.150 upper=2.150 effort=10 velocity=100 -> lower=-2.15 upper=2.15 effort=10 velocity=100; origin xyz=0 0 0.165 rpy=0 0 0 -> xyz=0 0 0.164999999999939 rpy=0 0 0
- joint moveo_joint3: limit lower=-2.150 upper=2.150 effort=10 velocity=100 -> lower=-2.15 upper=2.15 effort=10 velocity=100
- joint moveo_joint5: axis -0.99935 -0.035919 0 -> -0.99935 -0.035911 -0.00011484; limit lower=-2.150 upper=2.150 effort=10 velocity=100 -> lower=-1.4677 upper=1.9495 effort=10 velocity=100
- joint moveo_nozzle_joint: origin xyz=-0.013528 0.072912 0.10432 rpy=1.5418 0 0.035926 -> xyz=-0.00635 -0.034937 0.13566 rpy=3.1126 0 0.035926

Commit message: Auto_Rotate

File: moveo_urdf/urdf/moveo_urdf.urdf (robot description, URDF)
Before this commit: robot moveo_urdf, 8 links, 7 joints
Links:
- link base_link: mass 0.637576232475361 -> 0.637576232475362
- link moveo_link1: mass 4.20302329882691 -> 4.19319683049615
- link moveo_link2: mass 1.91858407297439 -> 1.92822525077319
- link moveo_link3: mass 0.648943927759347 -> 0.645102540582945
- link moveo_link4: mass 0.623350768745695 -> 0.361299996271292
- link moveo_link5: mass 0.157708115385714 -> 0.157708113676862
- link moveo_nozzle_link: mass 0.560923247976437 -> 0.551332467270815
Joints:
- joint moveo_joint2: axis -0.999386785928715 -0.0350150269323535 0 -> -0.99939 -0.035015 0; origin xyz=0 0 0.164999999999939 rpy=0 0 0 -> xyz=0 0 0.165 rpy=0 0 0
- joint moveo_joint4: limit lower=-3.1416 upper=3.1416 effort=10 velocity=100 -> lower=-1.3745 upper=4.5161 effort=10 velocity=100
- joint moveo_nozzle_joint: origin xyz=-0.00635 -0.034937 0.13566 rpy=3.1126 0 0.035926 -> xyz=-0.0094995 -0.039186 0.15124 rpy=-3.1401 0 0.035926

Commit message: cura_fix_moveo_fix

File: moveo_urdf/urdf/moveo_urdf.urdf (robot description, URDF)
Before this commit: robot moveo_urdf, 8 links, 7 joints
Links:
- link base_link: mass 0.637576232475362 -> 1.69354568563049
- link moveo_link1: mass 4.19319683049615 -> 4.17418410914588
- link moveo_link2: mass 1.92822525077319 -> 1.88123214398999
- link moveo_link3: mass 0.645102540582945 -> 0.612824408729849
- link moveo_link4: mass 0.361299996271292 -> 0.360582345944525
- link moveo_link5: mass 0.157708113676862 -> 0.156134491837058
- link moveo_nozzle_link: mass 0.551332467270815 -> 0.55163957172068
Joints:
- joint moveo_joint1: limit lower=-2.15 upper=2.15 effort=10 velocity=100 -> lower=-3.14159 upper=3.14159 effort=10 velocity=100; origin xyz=0 0 0.0665 rpy=0 0 0 -> xyz=0 0 0.1515 rpy=0 0 0; type revolute -> continuous
- joint moveo_joint2: axis -0.99939 -0.035015 0 -> -1 0 0
- joint moveo_joint3: axis -0.99939 -0.035015 0 -> -1 0 0; origin xyz=0.00099794 7.6228E-05 0.22112 rpy=0 0 0 -> xyz=0.001 6.9184E-05 0.22112 rpy=0 0 0
- joint moveo_joint4: axis 0.00023378 -0.0066725 0.99998 -> 0 -0.0066766 0.99998; origin xyz=2.9924E-05 -0.00085408 0.128 rpy=0 0 0 -> xyz=0 -0.0008546 0.128 rpy=0 0 0
- joint moveo_joint5: axis -0.99935 -0.035911 -0.00011484 -> -1 -0.00090423 0; origin xyz=2.2209E-05 -0.00063389 0.094998 rpy=0 0 0 -> xyz=0 -0.00063427 0.094998 rpy=0 0 0
- joint moveo_nozzle_joint: origin xyz=-0.0094995 -0.039186 0.15124 rpy=-3.1401 0 0.035926 -> xyz=-0.010865 -0.039338 0.15111 rpy=-3.1368 0 0.00090423

Commit message: add_alanboy's_code

File: moveo_urdf/urdf/moveo_urdf.urdf (robot description, URDF)
Before this commit: robot moveo_urdf, 8 links, 7 joints
Links:
- link base_link: mass 1.69354568563049 -> 0.637576232475362
- link moveo_link1: mass 4.17418410914588 -> 4.19319683049615
- link moveo_link2: mass 1.88123214398999 -> 1.92822525077319
- link moveo_link3: mass 0.612824408729849 -> 0.645102540582945
- link moveo_link4: mass 0.360582345944525 -> 0.361299996271292
- link moveo_link5: mass 0.156134491837058 -> 0.157708113676862
- link moveo_nozzle_link: mass 0.55163957172068 -> 0.551332467270815
Joints:
- joint moveo_joint1: limit lower=-3.14159 upper=3.14159 effort=10 velocity=100 -> lower=-2.15 upper=2.15 effort=10 velocity=100; origin xyz=0 0 0.1515 rpy=0 0 0 -> xyz=0 0 0.0665 rpy=0 0 0; type continuous -> revolute
- joint moveo_joint2: axis -1 0 0 -> -0.99939 -0.035015 0; limit lower=-1 upper=2.15 effort=10 velocity=100 -> lower=-2.15 upper=2.15 effort=10 velocity=100
- joint moveo_joint3: axis -1 0 0 -> -0.99939 -0.035015 0; limit lower=0 upper=2.15 effort=10 velocity=100 -> lower=-2.15 upper=2.15 effort=10 velocity=100; origin xyz=0.001 6.9184E-05 0.22112 rpy=0 0 0 -> xyz=0.00099794 7.6228E-05 0.22112 rpy=0 0 0
- joint moveo_joint4: axis 0 -0.0066766 0.99998 -> 0.00023378 -0.0066725 0.99998; origin xyz=0 -0.0008546 0.128 rpy=0 0 0 -> xyz=2.9924E-05 -0.00085408 0.128 rpy=0 0 0
- joint moveo_joint5: axis -1 -0.00090423 0 -> -0.99935 -0.035911 -0.00011484; origin xyz=0 -0.00063427 0.094998 rpy=0 0 0 -> xyz=2.2209E-05 -0.00063389 0.094998 rpy=0 0 0
- joint moveo_nozzle_joint: origin xyz=-0.010865 -0.039338 0.15111 rpy=-3.1368 0 0.00090423 -> xyz=-0.0094995 -0.039186 0.15124 rpy=-3.1401 0 0.035926

File: moveo_urdf/urdf/moveo_urdf1.urdf (robot description, URDF)
Before this commit: robot moveo_urdf, 8 links, 7 joints
Links:
- link base_link: mass 1.69354568563049 -> 0.637576232475362
- link moveo_link1: mass 4.17418410914588 -> 4.19319683049615
- link moveo_link2: mass 1.88123214398999 -> 1.92822525077319
- link moveo_link3: mass 0.612824408729849 -> 0.645102540582945
- link moveo_link4: mass 0.360582345944525 -> 0.361299996271292
- link moveo_link5: mass 0.156134491837058 -> 0.157708113676862
- link moveo_nozzle_link: mass 0.55163957172068 -> 0.551332467270815
Joints:
- joint moveo_joint1: limit lower=-3.14159 upper=3.14159 effort=10 velocity=100 -> lower=-2.15 upper=2.15 effort=10 velocity=100; origin xyz=0 0 0.1515 rpy=0 0 0 -> xyz=0 0 0.0665 rpy=0 0 0; type continuous -> revolute
- joint moveo_joint2: axis -1 0 0 -> -0.99939 -0.035015 0; limit lower=-1 upper=2.15 effort=10 velocity=100 -> lower=-2.15 upper=2.15 effort=10 velocity=100
- joint moveo_joint3: axis -1 0 0 -> -0.99939 -0.035015 0; limit lower=0 upper=2.15 effort=10 velocity=100 -> lower=-2.15 upper=2.15 effort=10 velocity=100; origin xyz=0.001 6.9184E-05 0.22112 rpy=0 0 0 -> xyz=0.00099794 7.6228E-05 0.22112 rpy=0 0 0
- joint moveo_joint4: axis 0 -0.0066766 0.99998 -> 0.00023378 -0.0066725 0.99998; origin xyz=0 -0.0008546 0.128 rpy=0 0 0 -> xyz=2.9924E-05 -0.00085408 0.128 rpy=0 0 0
- joint moveo_joint5: axis -1 -0.00090423 0 -> -0.99935 -0.035911 -0.00011484; origin xyz=0 -0.00063427 0.094998 rpy=0 0 0 -> xyz=2.2209E-05 -0.00063389 0.094998 rpy=0 0 0
- joint moveo_nozzle_joint: origin xyz=-0.010865 -0.039338 0.15111 rpy=-3.1368 0 0.00090423 -> xyz=-0.0094995 -0.039186 0.15124 rpy=-3.1401 0 0.035926

File: moveo_urdf/urdf/moveo_urdf2.urdf (robot description, URDF)
Before this commit: robot moveo_urdf, 8 links, 7 joints
Links:
- link base_link: mass 1.69354568563049 -> 0.637576232475362
- link moveo_link1: mass 4.17418410914588 -> 4.19319683049615
- link moveo_link2: mass 1.88123214398999 -> 1.92822525077319
- link moveo_link3: mass 0.612824408729849 -> 0.645102540582945
- link moveo_link4: mass 0.360582345944525 -> 0.361299996271292
- link moveo_link5: mass 0.156134491837058 -> 0.157708113676862
- link moveo_nozzle_link: mass 0.55163957172068 -> 0.551332467270815
Joints:
- joint moveo_joint1: limit lower=-3.14159 upper=3.14159 effort=10 velocity=100 -> lower=-2.15 upper=2.15 effort=10 velocity=100; origin xyz=0 0 0.1515 rpy=0 0 0 -> xyz=0 0 0.0665 rpy=0 0 0; type continuous -> revolute
- joint moveo_joint2: axis -1 0 0 -> -0.99939 -0.035015 0; limit lower=-1 upper=2.15 effort=10 velocity=100 -> lower=-2.15 upper=2.15 effort=10 velocity=100
- joint moveo_joint3: axis -1 0 0 -> -0.99939 -0.035015 0; limit lower=0 upper=2.15 effort=10 velocity=100 -> lower=-2.15 upper=2.15 effort=10 velocity=100; origin xyz=0.001 6.9184E-05 0.22112 rpy=0 0 0 -> xyz=0.00099794 7.6228E-05 0.22112 rpy=0 0 0
- joint moveo_joint4: axis 0 -0.0066766 0.99998 -> 0.00023378 -0.0066725 0.99998; origin xyz=0 -0.0008546 0.128 rpy=0 0 0 -> xyz=2.9924E-05 -0.00085408 0.128 rpy=0 0 0
- joint moveo_joint5: axis -1 -0.00090423 0 -> -0.99935 -0.035911 -0.00011484; origin xyz=0 -0.00063427 0.094998 rpy=0 0 0 -> xyz=2.2209E-05 -0.00063389 0.094998 rpy=0 0 0
- joint moveo_nozzle_joint: origin xyz=-0.010865 -0.039338 0.15111 rpy=-3.1368 0 0.00090423 -> xyz=-0.0094995 -0.039186 0.15124 rpy=-3.1401 0 0.035926

Commit message: link_cura_and_gcode_translation

File: moveo_urdf/urdf/moveo_urdf.urdf (robot description, URDF)
Before this commit: robot moveo_urdf, 8 links, 7 joints
Links:
- link base_link: mass 0.637576232475362 -> 1.69354568563049
- link moveo_link1: mass 4.19319683049615 -> 4.17418410914588
- link moveo_link2: mass 1.92822525077319 -> 1.88123214398999
- link moveo_link3: mass 0.645102540582945 -> 0.612824408729849
- link moveo_link4: mass 0.361299996271292 -> 0.360582345944525
- link moveo_link5: mass 0.157708113676862 -> 0.156134491837058
- link moveo_nozzle_link: mass 0.551332467270815 -> 0.55163957172068
Joints:
- joint moveo_joint1: limit lower=-2.15 upper=2.15 effort=10 velocity=100 -> lower=-3.14159 upper=3.14159 effort=10 velocity=100; origin xyz=0 0 0.0665 rpy=0 0 0 -> xyz=0 0 0.1515 rpy=0 0 0; type revolute -> continuous
- joint moveo_joint2: axis -0.99939 -0.035015 0 -> -1 0 0; limit lower=-2.15 upper=2.15 effort=10 velocity=100 -> lower=-1 upper=2.15 effort=10 velocity=100
- joint moveo_joint3: axis -0.99939 -0.035015 0 -> -1 0 0; limit lower=-2.15 upper=2.15 effort=10 velocity=100 -> lower=0 upper=2.15 effort=10 velocity=100; origin xyz=0.00099794 7.6228E-05 0.22112 rpy=0 0 0 -> xyz=0.001 6.9184E-05 0.22112 rpy=0 0 0
- joint moveo_joint4: axis 0.00023378 -0.0066725 0.99998 -> 0 -0.0066766 0.99998; origin xyz=2.9924E-05 -0.00085408 0.128 rpy=0 0 0 -> xyz=0 -0.0008546 0.128 rpy=0 0 0
- joint moveo_joint5: axis -0.99935 -0.035911 -0.00011484 -> -1 -0.00090423 0; origin xyz=2.2209E-05 -0.00063389 0.094998 rpy=0 0 0 -> xyz=0 -0.00063427 0.094998 rpy=0 0 0
- joint moveo_nozzle_joint: origin xyz=-0.0094995 -0.039186 0.15124 rpy=-3.1401 0 0.035926 -> xyz=-0.010865 -0.039338 0.15111 rpy=-3.1368 0 0.00090423

File: moveo_urdf/urdf/moveo_urdf1.urdf (robot description, URDF)
Before this commit: robot moveo_urdf, 8 links, 7 joints
Links:
- link base_link: mass 0.637576232475362 -> 1.69354568563049
- link moveo_link1: mass 4.19319683049615 -> 4.17418410914588
- link moveo_link2: mass 1.92822525077319 -> 1.88123214398999
- link moveo_link3: mass 0.645102540582945 -> 0.612824408729849
- link moveo_link4: mass 0.361299996271292 -> 0.360582345944525
- link moveo_link5: mass 0.157708113676862 -> 0.156134491837058
- link moveo_nozzle_link: mass 0.551332467270815 -> 0.55163957172068
Joints:
- joint moveo_joint1: limit lower=-2.15 upper=2.15 effort=10 velocity=100 -> lower=-3.14159 upper=3.14159 effort=10 velocity=100; origin xyz=0 0 0.0665 rpy=0 0 0 -> xyz=0 0 0.1515 rpy=0 0 0; type revolute -> continuous
- joint moveo_joint2: axis -0.99939 -0.035015 0 -> -1 0 0; limit lower=-2.15 upper=2.15 effort=10 velocity=100 -> lower=-1 upper=2.15 effort=10 velocity=100
- joint moveo_joint3: axis -0.99939 -0.035015 0 -> -1 0 0; limit lower=-2.15 upper=2.15 effort=10 velocity=100 -> lower=0 upper=2.15 effort=10 velocity=100; origin xyz=0.00099794 7.6228E-05 0.22112 rpy=0 0 0 -> xyz=0.001 6.9184E-05 0.22112 rpy=0 0 0
- joint moveo_joint4: axis 0.00023378 -0.0066725 0.99998 -> 0 -0.0066766 0.99998; origin xyz=2.9924E-05 -0.00085408 0.128 rpy=0 0 0 -> xyz=0 -0.0008546 0.128 rpy=0 0 0
- joint moveo_joint5: axis -0.99935 -0.035911 -0.00011484 -> -1 -0.00090423 0; origin xyz=2.2209E-05 -0.00063389 0.094998 rpy=0 0 0 -> xyz=0 -0.00063427 0.094998 rpy=0 0 0
- joint moveo_nozzle_joint: origin xyz=-0.0094995 -0.039186 0.15124 rpy=-3.1401 0 0.035926 -> xyz=-0.010865 -0.039338 0.15111 rpy=-3.1368 0 0.00090423

File: moveo_urdf/urdf/moveo_urdf2.urdf (robot description, URDF)
Before this commit: robot moveo_urdf, 8 links, 7 joints
Links:
- link base_link: mass 0.637576232475362 -> 1.69354568563049
- link moveo_link1: mass 4.19319683049615 -> 4.17418410914588
- link moveo_link2: mass 1.92822525077319 -> 1.88123214398999
- link moveo_link3: mass 0.645102540582945 -> 0.612824408729849
- link moveo_link4: mass 0.361299996271292 -> 0.360582345944525
- link moveo_link5: mass 0.157708113676862 -> 0.156134491837058
- link moveo_nozzle_link: mass 0.551332467270815 -> 0.55163957172068
Joints:
- joint moveo_joint1: limit lower=-2.15 upper=2.15 effort=10 velocity=100 -> lower=-3.14159 upper=3.14159 effort=10 velocity=100; origin xyz=0 0 0.0665 rpy=0 0 0 -> xyz=0 0 0.1515 rpy=0 0 0; type revolute -> continuous
- joint moveo_joint2: axis -0.99939 -0.035015 0 -> -1 0 0; limit lower=-2.15 upper=2.15 effort=10 velocity=100 -> lower=-1 upper=2.15 effort=10 velocity=100
- joint moveo_joint3: axis -0.99939 -0.035015 0 -> -1 0 0; limit lower=-2.15 upper=2.15 effort=10 velocity=100 -> lower=0 upper=2.15 effort=10 velocity=100; origin xyz=0.00099794 7.6228E-05 0.22112 rpy=0 0 0 -> xyz=0.001 6.9184E-05 0.22112 rpy=0 0 0
- joint moveo_joint4: axis 0.00023378 -0.0066725 0.99998 -> 0 -0.0066766 0.99998; origin xyz=2.9924E-05 -0.00085408 0.128 rpy=0 0 0 -> xyz=0 -0.0008546 0.128 rpy=0 0 0
- joint moveo_joint5: axis -0.99935 -0.035911 -0.00011484 -> -1 -0.00090423 0; origin xyz=2.2209E-05 -0.00063389 0.094998 rpy=0 0 0 -> xyz=0 -0.00063427 0.094998 rpy=0 0 0
- joint moveo_nozzle_joint: origin xyz=-0.0094995 -0.039186 0.15124 rpy=-3.1401 0 0.035926 -> xyz=-0.010865 -0.039338 0.15111 rpy=-3.1368 0 0.00090423
