Commit message: fix_IK_bug_and_change_URDF

File: moveo_urdf/urdf/moveo_urdf.urdf (robot description, URDF)
Before this commit: robot moveo_urdf, 8 links, 7 joints
Links:
- link base_link: mass 1.69354568563049 -> 2.57069193907154
- link moveo_link1: mass 4.17418410914588 -> 4.15952822957478
- link moveo_link2: mass 1.88123214398999 -> 1.8480863757448
- link moveo_link3: mass 0.612824408729849 -> 0.617310670458712
- link moveo_link4: mass 0.360582345944525 -> 0.346469873235592
- link moveo_link5: mass 0.156134491837058 -> 0.156134490695851
- link moveo_nozzle_link: mass 0.55163957172068 -> 0.571607414522843
Joints:
- joint moveo_joint1: origin xyz=0 0 0.1515 rpy=0 0 0 -> xyz=0 0 0.1715 rpy=0 0 0
- joint moveo_joint2: origin xyz=0 0 0.165 rpy=0 0 0 -> xyz=0 0 0.165000000000003 rpy=0 0 0
- joint moveo_joint3: origin xyz=0.001 6.9184E-05 0.22112 rpy=0 0 0 -> xyz=0.001 0 0.22112 rpy=0 0 0
- joint moveo_joint4: axis 0 -0.0066766 0.99998 -> 0 0 1; origin xyz=0 -0.0008546 0.128 rpy=0 0 0 -> xyz=0 0 0.1275 rpy=0 0 0
- joint moveo_joint5: axis -1 -0.00090423 0 -> 1 0 0; origin xyz=0 -0.00063427 0.094998 rpy=0 0 0 -> xyz=0 0.0001353 0.096 rpy=0 0 0
- joint moveo_nozzle_joint: origin xyz=-0.010865 -0.039338 0.15111 rpy=-3.1368 0 0.00090423 -> xyz=-0.0109 -0.0386 0.1513 rpy=-3.14159265358979 0 0

File: moveo_urdf/urdf/moveo_urdf1.urdf (robot description, URDF)
Before this commit: robot moveo_urdf, 8 links, 7 joints
Links:
- link base_link: mass 1.69354568563049 -> 2.57069193907154
- link moveo_link1: mass 4.17418410914588 -> 4.15952822957478
- link moveo_link2: mass 1.88123214398999 -> 1.8480863757448
- link moveo_link3: mass 0.612824408729849 -> 0.617310670458712
- link moveo_link4: mass 0.360582345944525 -> 0.346469873235592
- link moveo_link5: mass 0.156134491837058 -> 0.156134490695851
- link moveo_nozzle_link: mass 0.55163957172068 -> 0.571607414522843
Joints:
- joint moveo_joint1: origin xyz=0 0 0.1515 rpy=0 0 0 -> xyz=0 0 0.1715 rpy=0 0 0
- joint moveo_joint2: origin xyz=0 0 0.165 rpy=0 0 0 -> xyz=0 0 0.165000000000003 rpy=0 0 0
- joint moveo_joint3: origin xyz=0.001 6.9184E-05 0.22112 rpy=0 0 0 -> xyz=0.001 0 0.22112 rpy=0 0 0
- joint moveo_joint4: axis 0 -0.0066766 0.99998 -> 0 0 1; origin xyz=0 -0.0008546 0.128 rpy=0 0 0 -> xyz=0 0 0.1275 rpy=0 0 0
- joint moveo_joint5: axis -1 -0.00090423 0 -> 1 0 0; origin xyz=0 -0.00063427 0.094998 rpy=0 0 0 -> xyz=0 0.0001353 0.096 rpy=0 0 0
- joint moveo_nozzle_joint: origin xyz=-0.010865 -0.039338 0.15111 rpy=-3.1368 0 0.00090423 -> xyz=-0.0109 -0.0386 0.1513 rpy=-3.14159265358979 0 0

File: moveo_urdf/urdf/moveo_urdf2.urdf (robot description, URDF)
Before this commit: robot moveo_urdf, 8 links, 7 joints
Links:
- link base_link: mass 1.69354568563049 -> 2.57069193907154
- link moveo_link1: mass 4.17418410914588 -> 4.15952822957478
- link moveo_link2: mass 1.88123214398999 -> 1.8480863757448
- link moveo_link3: mass 0.612824408729849 -> 0.617310670458712
- link moveo_link4: mass 0.360582345944525 -> 0.346469873235592
- link moveo_link5: mass 0.156134491837058 -> 0.156134490695851
- link moveo_nozzle_link: mass 0.55163957172068 -> 0.571607414522843
Joints:
- joint moveo_joint1: origin xyz=0 0 0.1515 rpy=0 0 0 -> xyz=0 0 0.1715 rpy=0 0 0
- joint moveo_joint2: origin xyz=0 0 0.165 rpy=0 0 0 -> xyz=0 0 0.165000000000003 rpy=0 0 0
- joint moveo_joint3: origin xyz=0.001 6.9184E-05 0.22112 rpy=0 0 0 -> xyz=0.001 0 0.22112 rpy=0 0 0
- joint moveo_joint4: axis 0 -0.0066766 0.99998 -> 0 0 1; limit lower=3.05433 upper=3.22886 effort=10 velocity=100 -> lower=3.0543 upper=3.2289 effort=10 velocity=100; origin xyz=0 -0.0008546 0.128 rpy=0 0 0 -> xyz=0 0 0.1275 rpy=0 0 0
- joint moveo_joint5: axis -1 -0.00090423 0 -> 1 0 0; origin xyz=0 -0.00063427 0.094998 rpy=0 0 0 -> xyz=0 0.0001353 0.096 rpy=0 0 0
- joint moveo_nozzle_joint: origin xyz=-0.010865 -0.039338 0.15111 rpy=-3.1368 0 0.00090423 -> xyz=-0.0109 -0.0386 0.1513 rpy=-3.14159265358979 0 0

Commit message: fix_area_check_and_IK_first_point_bug

File: moveo_urdf/urdf/moveo_urdf.urdf (robot description, URDF)
Before this commit: robot moveo_urdf, 8 links, 7 joints
Links:
- link moveo_link2: mass 1.8480863757448 -> 1.84808635348241
- link moveo_link3: mass 0.617310670458712 -> 0.617310670458713
- link moveo_link4: mass 0.346469873235592 -> 0.346469873235588
- link moveo_link5: mass 0.156134490695851 -> 0.156134490708815
- link moveo_nozzle_link: mass 0.571607414522843 -> 0.571607414496871
Joints:
- joint moveo_joint2: origin xyz=0 0 0.165000000000003 rpy=0 0 0 -> xyz=0 0 0.165 rpy=0 0 0
- joint moveo_joint5: axis 1 0 0 -> -1 0 0; origin xyz=0 0.0001353 0.096 rpy=0 0 0 -> xyz=0 -0.000135303178896679 0.0960000000083613 rpy=0 0 0
- joint moveo_nozzle_joint: origin xyz=-0.0109 -0.0386 0.1513 rpy=-3.14159265358979 0 0 -> xyz=-0.0109 -0.0386000000000001 0.1513 rpy=-3.14159265358979 0 0

File: moveo_urdf/urdf/moveo_urdf1.urdf (robot description, URDF)
Before this commit: robot moveo_urdf, 8 links, 7 joints
Links:
- link moveo_link2: mass 1.8480863757448 -> 1.84808635348241
- link moveo_link3: mass 0.617310670458712 -> 0.617310670458713
- link moveo_link4: mass 0.346469873235592 -> 0.346469873235588
- link moveo_link5: mass 0.156134490695851 -> 0.156134490708815
- link moveo_nozzle_link: mass 0.571607414522843 -> 0.571607414496871
Joints:
- joint moveo_joint2: origin xyz=0 0 0.165000000000003 rpy=0 0 0 -> xyz=0 0 0.165 rpy=0 0 0
- joint moveo_joint5: axis 1 0 0 -> -1 0 0; origin xyz=0 0.0001353 0.096 rpy=0 0 0 -> xyz=0 -0.000135303178896679 0.0960000000083613 rpy=0 0 0
- joint moveo_nozzle_joint: origin xyz=-0.0109 -0.0386 0.1513 rpy=-3.14159265358979 0 0 -> xyz=-0.0109 -0.0386000000000001 0.1513 rpy=-3.14159265358979 0 0

File: moveo_urdf/urdf/moveo_urdf2.urdf (robot description, URDF)
Before this commit: robot moveo_urdf, 8 links, 7 joints
Links:
- link moveo_link2: mass 1.8480863757448 -> 1.84808635348241
- link moveo_link3: mass 0.617310670458712 -> 0.617310670458713
- link moveo_link4: mass 0.346469873235592 -> 0.346469873235588
- link moveo_link5: mass 0.156134490695851 -> 0.156134490708815
- link moveo_nozzle_link: mass 0.571607414522843 -> 0.571607414496871
Joints:
- joint moveo_joint2: origin xyz=0 0 0.165000000000003 rpy=0 0 0 -> xyz=0 0 0.165 rpy=0 0 0
- joint moveo_joint5: axis 1 0 0 -> -1 0 0; origin xyz=0 0.0001353 0.096 rpy=0 0 0 -> xyz=0 -0.000135303178896679 0.0960000000083613 rpy=0 0 0
- joint moveo_nozzle_joint: origin xyz=-0.0109 -0.0386 0.1513 rpy=-3.14159265358979 0 0 -> xyz=-0.0109 -0.0386000000000001 0.1513 rpy=-3.14159265358979 0 0
